File: intro-pcb.kicad_pcb (KiCad board)
At the start: 2 copper layers, 84.9 x 38.1 mm, 24 parts, among them SW1 SW_Push, U1 ATmega32U4-AU, Y1 Crystal_GND24_Small

Commit message: Generate Gerbers
Parts:
- added G***: LOGO, perce:logo_smallest, F.Cu at (-382.0, 49.5)
Routing:
- added copper zone on B.Cu, net GND
Other:
- board text added: "Hello World!"
- board text added: "Perce made this!!!"
